Commit message: wip

File: description/urdf/diffbot_description.urdf.xacro (robot description, xacro)
@@ -106,5 +106,5 @@
       </link>
           <!-- IMU Sensor -->
-    <link name="${prefix}imu">
+    <link name="${prefix}imu_link">
       <visual>
         <origin xyz="0 0 0" rpy="0 0 0"/>
@@ -117,5 +117,5 @@
     <joint name="${prefix}imu_joint" type="fixed">
       <parent link="${prefix}base_link"/>
-      <child link="${prefix}imu"/>
+      <child link="${prefix}imu_link"/>
       <origin xyz="0 0 ${base_height - imu_height}" rpy="0 0 0"/>
     </joint>

Commit message: Robot Navigating much better. Still has slam issues

File: description/urdf/diffbot_description.urdf.xacro (robot description, xacro)
@@ -36,8 +36,9 @@
       </inertial>
     </link>
+    <!-- left wheel Joint -->
     <joint name="${prefix}left_wheel_joint" type="continuous">
       <parent link="${prefix}base_link"/>
       <child link="${prefix}left_wheel"/>
-      <origin xyz="0 ${base_width/2} 0" rpy="0 0 0"/>
+      <origin xyz="0.02 ${base_width/2} 0" rpy="0 0 0"/>
       <axis xyz="0 1 0"/>
       <dynamics damping="0.2"/>
@@ -74,8 +75,9 @@
         </inertial>
       </link>
+    <!-- right wheel Joint -->
     <joint name="${prefix}right_wheel_joint" type="continuous">
       <parent link="${prefix}base_link"/>
       <child link="${prefix}right_wheel"/>
-      <origin xyz="0 -${base_width/2} 0" rpy="0 0 0"/>
+      <origin xyz="0.02 -${base_width/2} 0" rpy="0 0 0"/>
       <axis xyz="0 1 0"/>
       <dynamics damping="0.2"/>
@@ -118,5 +120,5 @@
       <parent link="${prefix}base_link"/>
       <child link="${prefix}imu_link"/>
-      <origin xyz="0 0 ${base_height - imu_height}" rpy="0 0 0"/>
+      <origin xyz="0.02 0 ${base_height - imu_height}" rpy="0 0 0"/>
     </joint>
           <!-- Lidar Sensor -->

Commit message: Small changes to improve odom

File: description/urdf/diffbot_description.urdf.xacro (robot description, xacro)
@@ -110,5 +110,5 @@
     <link name="${prefix}imu_link">
       <visual>
-        <origin xyz="0 0 0" rpy="0 0 0"/>
+        <origin xyz="0 0 0" rpy="0 ${pi} ${pi / 2}"/>
         <geometry>
           <box size="0.02 0.02 0.01"/>
@@ -137,4 +137,25 @@
       <origin xyz="0 0 ${base_height + 0.02}" rpy="0 0 ${PI}"/>
     </joint>
+    <!-- Camera -->
+    <link name="${prefix}camera_link">
+      <visual>
+        <origin xyz="0 0 0" rpy="0 0 0"/>
+        <geometry>
+          <box size="0.01 0.025 0.025"/>
+        </geometry>
+        <material name="green"/>
+      </visual>
+    </link>
+    <joint name="${prefix}camera_joint" type="fixed">
+      <parent link="${prefix}base_link"/>
+      <child link="${prefix}camera_link"/>
+      <origin xyz="0.08 0 ${base_height - imu_height}" rpy="0 0 0"/>
+    </joint>
+    <link name="${prefix}camera_link_optical"></link>
+    <joint name="${prefix}camera_optical_joint" type="fixed">
+      <parent link="${prefix}camera_link"/>
+      <child link="${prefix}camera_link_optical"/>
+      <origin xyz="0 0 0" rpy="${-PI/2} 0 ${-PI/2}"/>
+    </joint>
   </xacro:macro>
 </robot>

Commit message: Update urdf

File: description/urdf/diffbot_description.urdf.xacro (robot description, xacro)
@@ -120,5 +120,5 @@
       <parent link="${prefix}base_link"/>
       <child link="${prefix}imu_link"/>
-      <origin xyz="0.02 0 ${base_height - imu_height}" rpy="0 0 0"/>
+      <origin xyz="0.02 0.005 ${base_height - imu_height}" rpy="0 0 0"/>
     </joint>
           <!-- Lidar Sensor -->

Commit message: Params

File: description/urdf/diffbot_description.urdf.xacro (robot description, xacro)
@@ -11,5 +11,5 @@
   <xacro:property name="wheel_len" value="0.020" />
   <xacro:property name="wheel_radius" value="0.0175" />
-  <xacro:property name="imu_height" value="0.01" /> <!-- Height of IMU below top plate -->
+  <xacro:property name="imu_height" value="0.04" /> <!-- Height of IMU below top plate -->
   <!-- Base Link -->
   <link name="${prefix}base_link">
@@ -110,5 +110,5 @@
     <link name="${prefix}imu_link">
       <visual>
-        <origin xyz="0 0 0" rpy="0 ${pi} ${pi / 2}"/>
+        <origin xyz="0 0 0" rpy="0 0 0"/>
         <geometry>
           <box size="0.02 0.02 0.01"/>
@@ -120,5 +120,5 @@
       <parent link="${prefix}base_link"/>
       <child link="${prefix}imu_link"/>
-      <origin xyz="0.02 0.005 ${base_height - imu_height}" rpy="0 0 0"/>
+      <origin xyz="-0.02 0.01 ${base_height - imu_height}" rpy="0 0 ${PI}"/>
     </joint>
           <!-- Lidar Sensor -->
@@ -135,5 +135,5 @@
       <parent link="${prefix}base_link"/>
       <child link="${prefix}laser"/>
-      <origin xyz="0 0 ${base_height + 0.02}" rpy="0 0 ${PI}"/>
+      <origin xyz="0 0 ${base_height + 0.04}" rpy="0 0 ${PI}"/>
     </joint>
     <!-- Camera -->
