Commit message: wip

File: description/ros2_control/diffbot.ros2_control.xacro (robot description, xacro)
@@ -10,6 +10,6 @@
         <param name="bus_id">1</param> <!-- I2C Bus number (e.g., 1 for /dev/i2c-1) -->
         <param name="i2c_address">16</param> <!-- I2C Address of DFRobot board -->
-        <param name="max_rpm">75</param> <!-- I2C Address of DFRobot board -->
-        <param name="encoder_reduction_ratio">210</param> <!-- I2C Address of DFRobot board -->
+        <param name="max_rpm">75</param>
+        <param name="encoder_reduction_ratio">210</param>
         <param name="timeout_ms">1000</param>
         <param name="enc_counts_per_rev">3436</param>

File: description/urdf/diffbot_description.urdf.xacro (robot description, xacro)
@@ -43,4 +43,11 @@
       <dynamics damping="0.2"/>
     </joint>
+    <joint name="${prefix}base_footprint_joint" type="fixed">
+      <parent link="${prefix}base_link"/>
+      <child link="${prefix}base_footprint"/>
+      <origin xyz="0 0 0" rpy="0 0 0"/>
+    </joint>
+    <link name="base_footprint">
+    </link>
     <!-- left wheel Link -->
     <link name="${prefix}left_wheel">
@@ -126,5 +133,5 @@
       <parent link="${prefix}base_link"/>
       <child link="${prefix}laser"/>
-      <origin xyz="-0.01 0 ${base_height + 0.02}" rpy="0 0 ${PI}"/>
+      <origin xyz="0 0 ${base_height + 0.02}" rpy="0 0 ${PI}"/>
     </joint>
   </xacro:macro>
